Commit message: feat(kobuki_ws): Update kobuki description for gazebo world

File: kobuki_ws/src/kobuki_description/urdf/kobuki_gazebo.urdf.xacro (robot description, xacro)
@@ -40,131 +40,17 @@
 	      <always_on>1</always_on>
 	      <update_rate>50.0</update_rate>
-	      <visualize>true</visualize>
+	      <visualize>false</visualize>
 	      <contact>
-	        <collision>base_footprint_fixed_joint_lump__base_collision</collision>
+            <!-- Reference -->
+            <!-- https://answers.ros.org/question/334143/gazebo-bumper-sensor-states-msg-shows-no-output/ -->
+	        <collision>base_link_fixed_joint_lump__base_collision</collision>
 	      </contact>
+          <plugin name="plugin_name" filename="libgazebo_ros_bumper.so">
+            <ros>
+                <remapping>bumper_states:=/collision</remapping>
+            </ros>
+            <frame_name>world</frame_name>
+          </plugin>
 	    </sensor>
-	  </gazebo>
-	  <gazebo reference="cliff_sensor_left_link">
-	    <sensor type="ray" name="cliff_sensor_left">
-	      <always_on>true</always_on>
-	      <update_rate>50</update_rate>
-	      <visualize>true</visualize>
-	      <ray>
-	        <scan>
-	          <horizontal>
-	            <samples>50</samples>
-	            <resolution>1.0</resolution>
-	            <min_angle>-0.0436</min_angle>  <!-- -2.5 degree -->
-	            <max_angle>0.0436</max_angle> <!-- 2.5 degree -->
-	          </horizontal>
-			<!-- Can't use vertical rays until this bug is resolved -->
-			<!-- https://bitbucket.org/osrf/gazebo/issue/509/vertical-sensor-doesnt-works -->
-			<!-- <vertical> -->
-			<!--     <samples>50</samples> -->
-			<!--     <resolution>1.0</resolution> -->
-			<!--     <min_angle>-0.0436</min_angle>  -2.5 degree -->
-			<!--     <max_angle>0.0436</max_angle> 2.5 degree -->
-			<!-- </vertical> -->
-	        </scan>
-	        <range>
-	          <min>0.01</min>
-	          <max>0.15</max>
-	          <resolution>1.0</resolution>
-	        </range>
-	      </ray>
-	    </sensor>
-	  </gazebo>
-	  <gazebo reference="cliff_sensor_right_link">
-	    <sensor type="ray" name="cliff_sensor_right">
-	      <always_on>true</always_on>
-	      <update_rate>50</update_rate>
-	      <visualize>true</visualize>
-	      <ray>
-	        <scan>
-	          <horizontal>
-	            <samples>50</samples>
-	            <resolution>1.0</resolution>
-	            <min_angle>-0.0436</min_angle>  <!-- -2.5 degree -->
-	            <max_angle>0.0436</max_angle> <!-- 2.5 degree -->
-	          </horizontal>
-			<!-- Can't use vertical rays until this bug is resolved -->
-			<!-- https://bitbucket.org/osrf/gazebo/issue/509/vertical-sensor-doesnt-works -->
-			<!-- <vertical> -->
-			<!--     <samples>50</samples> -->
-			<!--     <resolution>1.0</resolution> -->
-			<!--     <min_angle>-0.0436</min_angle>  -2.5 degree -->
-			<!--     <max_angle>0.0436</max_angle> 2.5 degree -->
-			<!-- </vertical> -->
-	        </scan>
-	        <range>
-	          <min>0.01</min>
-	          <max>0.15</max>
-	          <resolution>1.0</resolution>
-	        </range>
-	      </ray>
-	    </sensor>
-	  </gazebo>
-	  <gazebo reference="cliff_sensor_front_link">
-	    <sensor type="ray" name="cliff_sensor_front">
-	      <always_on>true</always_on>
-	      <update_rate>50</update_rate>
-	      <visualize>true</visualize>
-	      <ray>
-	        <scan>
-	          <horizontal>
-	            <samples>50</samples>
-	            <resolution>1.0</resolution>
-	            <min_angle>-0.0436</min_angle>  <!-- -2.5 degree -->
-	            <max_angle>0.0436</max_angle> <!-- 2.5 degree -->
-	          </horizontal>
-			<!-- Can't use vertical rays until this bug is resolved -->
-			<!-- https://bitbucket.org/osrf/gazebo/issue/509/vertical-sensor-doesnt-works -->
-			<!-- <vertical> -->
-			<!--     <samples>50</samples> -->
-			<!--     <resolution>1.0</resolution> -->
-			<!--     <min_angle>-0.0436</min_angle>  -2.5 degree -->
-			<!--     <max_angle>0.0436</max_angle> 2.5 degree -->
-			<!-- </vertical> -->
-	        </scan>
-	        <range>
-	          <min>0.01</min>
-	          <max>0.15</max>
-	          <resolution>1.0</resolution>
-	        </range>
-	      </ray>
-	    </sensor>
-	  </gazebo>
-	  <gazebo reference="gyro_link">
-	   <sensor type="imu" name="imu">
-        <plugin name="gazebo_ros_imu_controller" filename="libgazebo_ros_imu_sensor.so">
-          <ros>
-            <remapping>~/out:=/imu/data_raw</remapping>
-          </ros>
-          <output_type>sensor_msgs/msg/Imu</output_type>
-          <body_name>gyro_link</body_name>
-          <frame_name>gyro_link</frame_name>
-        </plugin>
-        <always_on>true</always_on>
-        <update_rate>50</update_rate>
-        <visualize>false</visualize>
-        <imu>
-          <noise>
-            <type>gaussian</type>
-	          <rate>
-	            <mean>0.0</mean>
-	            <stddev>${0.0014*0.0014}</stddev> <!-- 0.25 x 0.25 (deg/s) -->
-	            <bias_mean>0.0</bias_mean>
-	            <bias_stddev>0.0</bias_stddev>
-	          </rate>
-		        <accel> <!-- not used in the plugin and real robot, hence using tutorial values -->
-			        <mean>0.0</mean>
-			        <stddev>1.7e-2</stddev>
-			        <bias_mean>0.1</bias_mean>
-			        <bias_stddev>0.001</bias_stddev>
-		        </accel>
-          </noise>
-	      </imu>
-      </sensor>
 	  </gazebo>
 	  <gazebo>
